File: ThermistorComparator.sch (KiCad schematic (older format))
At the start: 20 parts, among them J1 i/o_unique, J2 i/o, J3 pwr_conn, U1 TLP171A, U12 LTC3637IMSE-PBF

Commit message: new
Parts:
- removed R2: 10k, Resistor_SMD:R_0603_1608Metric_Pad0.98x0.95mm_HandSolder, symbol Device:R
- added J4: UNIQUE_PWR_CONN, Connector_Molex:Molex_Micro-Fit_3.0_43045-0200_2x01_P3.00mm_Horizontal, symbol Connector_Generic:Conn_01x02
- D1: footprint (none) -> LHRE Footprint Library:SBR3U100LP7
- J1: value i/o_unique -> I/O; footprint Connector_Molex:Molex_Micro-Fit_3.0_43045-0200_2x01_P3.00mm_Horizontal -> Connector_Molex:Molex_Micro-Fit_3.0_43045-0400_2x02_P3.00mm_Horizontal; symbol Connector_Generic:Conn_01x02 -> Connector_Generic:Conn_01x04
- J2: value i/o -> UNIQUE_I/O; footprint Connector_Molex:Molex_Micro-Fit_3.0_43045-0200_2x01_P3.00mm_Horizontal -> Connector_Molex:Molex_Micro-Fit_3.0_43045-0410_2x02-1MP_P3.00mm_Horizontal; symbol Connector_Generic:Conn_01x02 -> Connector_Generic:Conn_01x04
- J3: value pwr_conn -> PWR_CONN
- R1: value 2.2k -> 1.8k
- U12: footprint (none) -> LHRE Footprint Library:LTC3637IMSE-PBF
Connections:
- net GND: now also J1.3 (Pin_3), J1.4 (Pin_4), J2.3 (Pin_3), J2.4 (Pin_4), J4.2 (Pin_2)
- net RUN: now also J4.1 (Pin_1)
Other:
- moved on the sheet: J3, R1, RV1, RV2, TP1, TP3, TP4, TP7, U1

Commit message: Add files via upload
Parts:
- removed C2: 100 uF, Capacitor_SMD:C_1210_3225Metric_Pad1.33x2.70mm_HandSolder, symbol Device:C
- removed J2: UNIQUE_I/O, Connector_Molex:Molex_Micro-Fit_3.0_43045-0410_2x02-1MP_P3.00mm_Horizontal, symbol Connector_Generic:Conn_01x04
- added C3, C5, C6: 100 uF, Capacitor_SMD:C_1210_3225Metric_Pad1.33x2.70mm_HandSolder, symbol Device:C
- added C4: 47pF, Capacitor_SMD:C_0603_1608Metric_Pad1.08x0.95mm_HandSolder, symbol Device:C
- added Cin2: 4.7 uF, Capacitor_SMD:C_2220_5650Metric_Pad1.97x5.40mm_HandSolder, symbol Device:C
- added D2: SBR3U100LP-7, LHRE Footprint Library:SBR3U100LP7, symbol SBR3U100LP-7:SBR3U100LP-7
- added J2: OUT, Connector_Molex:Molex_Micro-Fit_3.0_43045-0200_2x01_P3.00mm_Horizontal, symbol Connector_Generic:Conn_01x02
- added J3: UNIQUE_IN, Connector_Molex:Molex_Micro-Fit_3.0_43045-0210_2x01-1MP_P3.00mm_Horizontal, symbol Connector_Generic:Conn_01x02
- added J4: UNIQUE_OUT, Connector_Molex:Molex_Micro-Fit_3.0_43045-0210_2x01-1MP_P3.00mm_Horizontal, symbol Connector_Generic:Conn_01x02
- added L2: 10 uH, Inductor_SMD:L_Sumida_CDRH105RNP-100NC, symbol Device:L
- added R22: 255k, Resistor_SMD:R_1210_3225Metric_Pad1.30x2.65mm_HandSolder, symbol Device:R
- added R3: 3k, Resistor_SMD:R_0805_2012Metric_Pad1.20x1.40mm_HandSolder, symbol Device:R
- added RV3: 1.9k, Potentiometer_THT:Potentiometer_Bourns_3299P_Horizontal, symbol Device:R_Potentiometer
- added RV4: 1.1k, Potentiometer_THT:Potentiometer_Bourns_3299P_Horizontal, symbol Device:R_Potentiometer
- added U8: LTC3637IMSE-PBF, LHRE Footprint Library:LTC3637IMSE-PBF, symbol 2023-01-15_21-00-20:LTC3637IMSE-PBF
- C1: renamed from C3; value 4.7pF -> 47pF; website (none) -> https://www.digikey.com/en/products/detail/vishay-vitramon/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
- C2: renamed from C1; digikey (none) -> https://www.digikey.com/en/products/detail/murata-electroni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
- J1: value I/O -> IN; footprint Connector_Molex:Molex_Micro-Fit_3.0_43045-0400_2x02_P3.00mm_Horizontal -> Connector_Molex:Molex_Micro-Fit_3.0_43045-0200_2x01_P3.00mm_Horizontal; symbol Connector_Generic:Conn_01x04 -> Connector_Generic:Conn_01x02
- J6: renamed from J4; footprint Connector_Molex:Molex_Micro-Fit_3.0_43045-0200_2x01_P3.00mm_Horizontal -> Connector_Molex:Molex_Micro-Fit_3.0_43045-0210_2x01-1MP_P3.00mm_Horizontal
- R1: renamed from R23; footprint Resistor_SMD:R_0603_1608Metric_Pad0.98x0.95mm_HandSolder -> Resistor_SMD:R_1210_3225Metric_Pad1.30x2.65mm_HandSolder; digikey (none) -> https://www.digikey.com/en/products/detail/panasonic-electr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
- R2: renamed from R1; value 1.8k -> 370; footprint Resistor_SMD:R_0603_1608Metric_Pad0.98x0.95mm_HandSolder -> Resistor_SMD:R_0805_2012Metric_Pad1.20x1.40mm_HandSolder; Description (none) -> Thin Film Resistors - SMD 370Ohm,0805,0.1%,25p pm,125mW,100V
- renumbered J3 to J5, TP7 to TP1, TP4 to TP2, TP1 to TP3, TP3 to TP4, U12 to U1, U1 to U2
Connections:
- net FAULT: now also J2.1 (Pin_1), J3.1 (Pin_1), J4.1 (Pin_1); no longer J1.2 (Pin_2)
- net GND: now also C2.2, D1.1 (A_1), D1.2 (A_2), D1.3 (A_3), D1.4 (A_4), J1.2 (Pin_2), C3.2, C4.2, C5.2, C6.2, Cin2.2, D2.1 (A_1), D2.2 (A_2), D2.3 (A_3), D2.4 (A_4), J2.2 (Pin_2), J3.2 (Pin_2), J4.2 (Pin_2), R22.2, RV4.2, U8.12 (OVLO), U8.16 (GND), U8.17 (GND), U8.6 (VPRG2), U8.8 (GND); no longer D1.5 (K), J1.3 (Pin_3), J1.4 (Pin_4)
- net IN+: now also RV3.2, RV4.1
- net RUN: now also Cin2.1, U8.14 (RUN), U8.3 (VIN)
- net V+: now also C3.1, C5.1, C6.1, L2.2, R3.2, RV3.1, U8.9 (VFB)
- net SIG renamed OUT
- net OUT: now also R3.1
- new net: D1.5 (K), L1.1, U1.1 (SW)
- new net: D2.5 (K), L2.1, U8.1 (SW)
- new net: C4.1, R22.1, U8.11 (ISET)
- new net prg1B: U8.10 (SS), U8.7 (VPRG1)
- no-connect marks 3 -> 6
Other:
- moved on the sheet: C1, C2, Cin1, D1, J5, J6, L1, R1, R2, RV1, RV2, TP1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
