File: ThermistorComparator.kicad_pcb (KiCad board)
At the start: 2 copper layers, 278 x 115 mm, 66 parts, among them J1 main/daisy_out, J2 Daisy_in, U1 TLP171A, U10 LM393M, U11 LM393M, U2 LM393M, U3 LM393M, U4 LM393M, U5 LM393M, U6 LM393M, U7 LM393M, U8 LM393M, U9 LM393M

Commit message: Add files via upload
Parts:
- removed the R2 at (-169.1, -358.2)
- removed TH19, TH20: 100k, Resistor_SMD:R_0603_1608Metric_Pad0.98x0.95mm_HandSolder
- removed TP1: Test_gnd, LHRE Footprint Library:Test_Point_Tiny
- removed TP2: Test_v+, LHRE Footprint Library:Test_Point_Tiny
- removed TP3: Test_sig, LHRE Footprint Library:Test_Point_Tiny
- removed TP4: Test_in+, LHRE Footprint Library:Test_Point_Tiny
- removed TP5: Test_t1, LHRE Footprint Library:Test_Point_Tiny
- removed TP6: Test_t15, LHRE Footprint Library:Test_Point_Tiny
- removed TP7: Test_fault, LHRE Footprint Library:Test_Point_Tiny
- removed TP8: Test_v-, LHRE Footprint Library:Test_Point_Tiny
- removed U10, U11, U9: LM393M, LHRE Footprint Library:SOIC127P599X175-8N
- removed the U2 at (-169.3, -328.9)
- added C1: 47pF, Capacitor_SMD:C_0603_1608Metric_Pad1.08x0.95mm_HandSolder, F.Cu at (215.0, 21.9)
- added C2: 100 uF, Capacitor_SMD:C_1210_3225Metric_Pad1.33x2.70mm_HandSolder, F.Cu at (228.0, 19.6)
- added C3: 100 uF, Capacitor_SMD:C_1210_3225Metric_Pad1.33x2.70mm_HandSolder, F.Cu at (224.6, 19.6)
- added C4: 47pF, Capacitor_SMD:C_0603_1608Metric_Pad1.08x0.95mm_HandSolder, B.Cu at (217.3, 70.9)
- added C5: 100 uF, Capacitor_SMD:C_1210_3225Metric_Pad1.33x2.70mm_HandSolder, B.Cu at (219.1, 56.9)
- added C6: 100 uF, Capacitor_SMD:C_1210_3225Metric_Pad1.33x2.70mm_HandSolder, B.Cu at (219.2, 60.2)
- added Cin1: 4.7 uF, Capacitor_SMD:C_2220_5650Metric_Pad1.97x5.40mm_HandSolder, F.Cu at (226.2, 12.4)
- added Cin2: 4.7 uF, Capacitor_SMD:C_2220_5650Metric_Pad1.97x5.40mm_HandSolder, B.Cu at (226.7, 58.5)
- added D2: SBR3U100LP-7, LHRE Footprint Library:SBR3U100LP7, B.Cu at (225.9, 64.3)
- added J3: UNIQUE_IN, Connector_Molex:Molex_Micro-Fit_3.0_43045-0210_2x01-1MP_P3.00mm_Horizontal, B.Cu at (23.7, 53.9)
- added J4: UNIQUE_OUT, Connector_Molex:Molex_Micro-Fit_3.0_43045-0210_2x01-1MP_P3.00mm_Horizontal, B.Cu at (36.0, 53.9)
- added J5: PWR_CONN, Connector_Molex:Molex_Micro-Fit_3.0_43045-0200_2x01_P3.00mm_Horizontal, F.Cu at (268.6, 19.9)
- added J6: UNIQUE_PWR_CONN, Connector_Molex:Molex_Micro-Fit_3.0_43045-0210_2x01-1MP_P3.00mm_Horizontal, F.Cu at (264.4, 51.5)
- added L1: 10 uH, Inductor_SMD:L_Sumida_CDRH105RNP-100NC, F.Cu at (234.9, 16.8)
- added L2: 10 uH, Inductor_SMD:L_Sumida_CDRH105RNP-100NC, B.Cu at (221.9, 50.0)
- added R1: 255k, Resistor_SMD:R_1210_3225Metric_Pad1.30x2.65mm_HandSolder, F.Cu at (217.6, 22.6)
- added RV3: 1.9k, Potentiometer_THT:Potentiometer_Bourns_3299P_Horizontal, B.Cu at (60.8, 43.8)
- added RV4: 1.1k, Potentiometer_THT:Potentiometer_Bourns_3299P_Horizontal, B.Cu at (50.6, 44.0)
- added U1: MSE_16A_ADI, LHRE Footprint Library:LTC3637IMSE-PBF, F.Cu at (215.7, 15.8)
- D1: value REM2-1212S -> SBR3U100LP-7; footprint Converter_DCDC:CONV_REM2-1212S -> LHRE Footprint Library:SBR3U100LP7
- J1: value main/daisy_out -> IN; footprint Connector_Molex:Molex_Micro-Fit_3.0_43045-0400_2x02_P3.00mm_Horizontal -> Connector_Molex:Molex_Micro-Fit_3.0_43045-0200_2x01_P3.00mm_Horizontal
- J2: value Daisy_in -> OUT; footprint Connector_Molex:Molex_Micro-Fit_3.0_43045-0400_2x02_P3.00mm_Horizontal -> Connector_Molex:Molex_Micro-Fit_3.0_43045-0200_2x01_P3.00mm_Horizontal
- R2: renamed from R1; value 5.5k -> 370; footprint Resistor_SMD:R_0603_1608Metric_Pad0.98x0.95mm_HandSolder -> Resistor_SMD:R_0805_2012Metric_Pad1.20x1.40mm_HandSolder
- R22: value 2k -> 255k; footprint Resistor_SMD:R_0805_2012Metric_Pad1.20x1.40mm_HandSolder -> Resistor_SMD:R_1210_3225Metric_Pad1.30x2.65mm_HandSolder; moved to B.Cu
- R3: value 2k -> 3k
- TH1, TH11, TH12, TH13, TH14, TH15, TH2, TH3, TH4, TH5: footprint Resistor_SMD:R_0603_1608Metric_Pad0.98x0.95mm_HandSolder -> Resistor_SMD:R_1206_3216Metric_Pad1.30x1.75mm_HandSolder
- TH10, TH16, TH17, TH18, TH6, TH7, TH8, TH9: value 100k -> 1k; footprint Resistor_SMD:R_0603_1608Metric_Pad0.98x0.95mm_HandSolder -> Resistor_SMD:R_1206_3216Metric_Pad1.30x1.75mm_HandSolder
- U3, U4, U5, U6, U7: value LM393M -> LMV339MX_NOPB; footprint LHRE Footprint Library:SOIC127P599X175-8N -> LHRE Footprint Library:SOIC127P600X175-14N; moved to B.Cu
- U8: value LM393M -> MSE_16A_ADI; footprint LHRE Footprint Library:SOIC127P599X175-8N -> LHRE Footprint Library:LTC3637IMSE-PBF; moved to B.Cu
- moved U4 604.3 mm to (262.9, 87.0), turned to 270 degrees
- moved U7 586.9 mm to (209.0, 104.0), turned to 270 degrees
- moved U8 574.7 mm to (223.5, 69.2), turned to 180 degrees
- moved U6 557.8 mm to (183.2, 90.5), turned to 270 degrees
- moved R2 547.6 mm to (198.7, 42.3), turned to 180 degrees
- moved U5 510.0 mm to (114.1, 89.0), turned to 270 degrees
- moved U3 492.1 mm to (69.9, 93.1), turned to 270 degrees
- moved TH18 489.3 mm to (281.7, 134.8), turned to 90 degrees
- moved TH7 488.9 mm to (91.6, 83.1), turned to 90 degrees
- moved R21 485.7 mm to (281.7, 130.3), turned to 90 degrees
- moved TH2 468.0 mm to (53.6, 83.1), turned to 90 degrees
- moved R9 456.9 mm to (281.5, 78.3), turned to 90 degrees
- moved R4 452.1 mm to (15.6, 78.3), turned to 90 degrees
- moved TH6 447.4 mm to (281.5, 82.9), turned to 90 degrees
- moved R16 439.5 mm to (205.6, 130.4), turned to 90 degrees
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- renumbered U1 to U2
Connections:
- D1 pad 1: +12V -> GND
- J1 pad 1: +12V -> /FAULT
- J2 pad 1: /SIG -> /FAULT
- J2 pad 2: IN+ -> GND
- R10 pad 1: V+ -> Net-(R10-Pad1)
- R10 pad 2: Net-(R10-Pad2) -> GND
- R11 pad 1: V+ -> Net-(R11-Pad1)
- R11 pad 2: Net-(R11-Pad2) -> GND
- R12 pad 1: V+ -> Net-(R12-Pad1)
- R12 pad 2: Net-(R12-Pad2) -> GND
- R13 pad 1: V+ -> Net-(R13-Pad1)
- R13 pad 2: Net-(R13-Pad2) -> GND
- R14 pad 1: V+ -> Net-(R14-Pad1)
- R14 pad 2: Net-(R14-Pad2) -> GND
- R15 pad 1: V+ -> Net-(R15-Pad1)
- R15 pad 2: Net-(R15-Pad2) -> GND
- R16 pad 1: V+ -> Net-(R16-Pad1)
- R16 pad 2: Net-(R16-Pad2) -> GND
- R17 pad 1: V+ -> Net-(R17-Pad1)
- R17 pad 2: Net-(R17-Pad2) -> GND
- R18 pad 1: V+ -> Net-(R18-Pad1)
- R18 pad 2: Net-(R18-Pad2) -> GND
- R19 pad 1: V+ -> Net-(R19-Pad1)
- R19 pad 2: Net-(R19-Pad2) -> GND
- R20 pad 1: V+ -> Net-(R20-Pad1)
- R20 pad 2: Net-(R20-Pad2) -> GND
- R21 pad 1: V+ -> Net-(R21-Pad1)
- R21 pad 2: Net-(R21-Pad2) -> GND
- R22 pad 1: V+ -> Net-(C4-Pad1)
- R22 pad 2: Net-(R22-Pad2) -> GND
- R3 pad 1: V+ -> /OUT
- R3 pad 2: Net-(R3-Pad2) -> V+
- R4 pad 1: V+ -> Net-(R4-Pad1)
- R4 pad 2: Net-(R4-Pad2) -> GND
- R5 pad 1: V+ -> Net-(R5-Pad1)
- R5 pad 2: Net-(R5-Pad2) -> GND
- R6 pad 1: V+ -> Net-(R6-Pad1)
- R6 pad 2: Net-(R6-Pad2) -> GND
- R7 pad 1: V+ -> Net-(R7-Pad1)
- R7 pad 2: Net-(R7-Pad2) -> GND
- R8 pad 1: V+ -> Net-(R8-Pad1)
- R8 pad 2: Net-(R8-Pad2) -> GND
- R9 pad 1: V+ -> Net-(R9-Pad1)
- R9 pad 2: Net-(R9-Pad2) -> GND
- RV2 pad 2: V- -> GND
- TH1 pad 1: V- -> V+
- TH1 pad 2: Net-(R3-Pad2) -> Net-(R4-Pad1)
- TH10 pad 1: V- -> V+
- TH10 pad 2: Net-(R12-Pad2) -> Net-(R13-Pad1)
- TH11 pad 1: V- -> V+
- TH11 pad 2: Net-(R13-Pad2) -> Net-(R14-Pad1)
- TH12 pad 1: V- -> V+
- TH12 pad 2: Net-(R14-Pad2) -> Net-(R15-Pad1)
- TH13 pad 1: V- -> V+
- TH13 pad 2: Net-(R15-Pad2) -> Net-(R16-Pad1)
- TH14 pad 1: V- -> V+
- TH14 pad 2: Net-(R16-Pad2) -> Net-(R17-Pad1)
- TH15 pad 1: V- -> V+
- TH15 pad 2: Net-(R17-Pad2) -> Net-(R18-Pad1)
- TH16 pad 1: V- -> V+
- TH16 pad 2: Net-(R18-Pad2) -> Net-(R19-Pad1)
- TH17 pad 1: V- -> V+
- TH17 pad 2: Net-(R19-Pad2) -> Net-(R20-Pad1)
- TH18 pad 1: V- -> V+
- TH18 pad 2: Net-(R20-Pad2) -> Net-(R21-Pad1)
- TH2 pad 1: V- -> V+
- TH2 pad 2: Net-(R4-Pad2) -> Net-(R5-Pad1)
- TH3 pad 1: V- -> V+
- TH3 pad 2: Net-(R5-Pad2) -> Net-(R6-Pad1)
- TH4 pad 1: V- -> V+
- TH4 pad 2: Net-(R6-Pad2) -> Net-(R7-Pad1)
- TH5 pad 1: V- -> V+
- TH5 pad 2: Net-(R7-Pad2) -> Net-(R8-Pad1)
- TH6 pad 1: V- -> V+
- TH6 pad 2: Net-(R8-Pad2) -> Net-(R9-Pad1)
- TH7 pad 1: V- -> V+
- TH7 pad 2: Net-(R9-Pad2) -> Net-(R10-Pad1)
- TH8 pad 1: V- -> V+
- TH8 pad 2: Net-(R10-Pad2) -> Net-(R11-Pad1)
- TH9 pad 1: V- -> V+
- TH9 pad 2: Net-(R11-Pad2) -> Net-(R12-Pad1)
- U2 pad 2: /SIG -> /OUT
- U3 pad 1: /SIG -> /OUT
- U3 pad 2: Net-(R9-Pad2) -> /OUT
- U3 pad 3: IN+ -> V+
- U3 pad 4: V- -> Net-(R4-Pad1)
- U3 pad 6: Net-(R4-Pad2) -> Net-(R5-Pad1)
- U3 pad 7: /SIG -> IN+
- U3 pad 8: V+ -> Net-(R6-Pad1)
- U4 pad 1: /SIG -> /OUT
- U4 pad 2: Net-(R10-Pad2) -> /OUT
- U4 pad 3: IN+ -> V+
- U4 pad 4: V- -> Net-(R8-Pad1)
- U4 pad 6: Net-(R5-Pad2) -> Net-(R9-Pad1)
- U4 pad 7: /SIG -> IN+
- U4 pad 8: V+ -> Net-(R9-Pad1)
- U5 pad 1: /SIG -> /OUT
- U5 pad 2: Net-(R11-Pad2) -> /OUT
- U5 pad 3: IN+ -> V+
- U5 pad 4: V- -> Net-(R10-Pad1)
- U5 pad 6: Net-(R6-Pad2) -> Net-(R11-Pad1)
- U5 pad 7: /SIG -> IN+
- U5 pad 8: V+ -> Net-(R12-Pad1)
- U6 pad 1: /SIG -> /OUT
- U6 pad 2: Net-(R12-Pad2) -> /OUT
- U6 pad 3: IN+ -> V+
- U6 pad 4: V- -> Net-(R14-Pad1)
- U6 pad 6: Net-(R7-Pad2) -> Net-(R15-Pad1)
- U6 pad 7: /SIG -> IN+
- U6 pad 8: V+ -> Net-(R16-Pad1)
- U7 pad 1: /SIG -> /OUT
- U7 pad 2: Net-(R18-Pad2) -> /OUT
- U7 pad 3: IN+ -> V+
- U7 pad 4: V- -> Net-(R18-Pad1)
- U7 pad 6: Net-(R13-Pad2) -> Net-(R19-Pad1)
- U7 pad 7: /SIG -> IN+
- U7 pad 8: V+ -> Net-(R20-Pad1)
- U8 pad 1: /SIG -> Net-(D2-Pad5)
- U8 pad 3: IN+ -> RUN
- U8 pad 5: IN+ -> Net-(U8-Pad5)
- U8 pad 6: Net-(R14-Pad2) -> GND
- U8 pad 7: /SIG -> prg1B
- U8 pad 8: V+ -> GND
Routing:
- net IN+: track 0.00 -> 387.3 mm, vias 0 -> 5
- net /OUT: track 0.00 -> 348.5 mm, vias 0 -> 7
- net GND: track 0.00 -> 234.3 mm, vias 0 -> 10
- net /FAULT: track 0.00 -> 213.8 mm, vias 0 -> 2
- net RUN: track 0.00 -> 122.2 mm, vias 0 -> 10
- net Net-(R21-Pad1): track 0.00 -> 89.3 mm, vias 0 -> 1
- net V+: track 0.00 -> 78.3 mm, vias 0 -> 34
- net Net-(R4-Pad1): track 0.00 -> 63.2 mm, vias 0 -> 1
- net Net-(R13-Pad1): track 0.00 -> 54.5 mm, vias 0 -> 1
- net Net-(R6-Pad1): track 0.00 -> 53.9 mm, vias 0 -> 1
- net Net-(R19-Pad1): track 0.00 -> 52.3 mm, vias 0 -> 1
- net Net-(R7-Pad1): track 0.00 -> 51.4 mm, vias 0 -> 1
- net Net-(R16-Pad1): track 0.00 -> 51.2 mm, vias 0 -> 1
- net Net-(R17-Pad1): track 0.00 -> 50.3 mm, vias 0 -> 1
- net Net-(R11-Pad1): track 0.00 -> 44.2 mm, vias 0 -> 1
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- added copper zone on B.Cu, net GND
- added copper zone on F.Cu, net GND
- added copper zone on F.Cu, net Net-(D1-Pad5)
- added copper zone on B.Cu, net Net-(D2-Pad5)
- added copper zone on B.Cu, net RUN
- added copper zone on F.Cu, net RUN
- added copper zone on B.Cu, net V+
- added copper zone on F.Cu, net V+
Other:
- board size 278 x 115 mm -> 278 x 145.4 mm
- net class Default: clearance 0.2 -> 0.153
- rule trace_clearance: 0.2 -> 0.153
- rule trace_min: 0.2 -> 0.155
- rule via_min_size: 0.4 -> 0.26
- board text added: "For Instructional Use Only."
- board text added: "SOLIDWORKS Educational Product."
- board text added: "YOU'RE HOT"
- board text added: "i*r"

Commit message: Add files via upload
Routing:
- net GND: track 234.3 -> 60.5 mm
- net V+: track 78.3 -> 46.4 mm
- net /FAULT: track 213.8 -> 215.4 mm
- net RUN: track 122.2 -> 122.6 mm, vias 10 -> 11
Other:
- outline, holes or cut-outs redrawn
